File: ngptv/ngptv.sch (EAGLE design)
At the start: 55 parts, among them J1 2013978-1, U1 ADV7533BCBZ-RL, U2 MIC5387-SG4YMT, U3 IP4786CZ32S, U4 TPS61240YFFR, U5 PCMF2HDMI2S, X1 SIT8021AI-J4-18S-12.000000E

Commit message: Updated sch
Parts:
- added R5: 0R, Seeed-Resistor:SMD-RES-0R-5%-1/16W(0402)
Connections:
- net N$1 renamed PVDD
- net N$15 renamed TXC_P
- net N$16 renamed TXC_N
- net N$17 renamed TX2_P
- net N$18 renamed TX2_N
- net N$19 renamed TX1_P
- net N$2 renamed A2VDD
- net N$20 renamed TX1_N
- net N$21 renamed TX0_P
- net N$22 renamed TX0_N
- net N$28 renamed AVDD
- net N$3 renamed DVDD
- net N$4 renamed V1P2
- net N$5 renamed V3P3
- net CEC_CLK: now also R5.2
- net GND: now also R5.1
Other:
- note added: "Bridge to disable CEC"
Changed lines of the file:
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@@
 <part name="SPDIF" library="testpad" library_urn="urn:adsk.eagle:library:385" deviceset="TP" device="TP10R" package3d_urn="urn:adsk.eagle:package:27959/1"/>
 <part name="GND23" library="supply1" library_urn="urn:adsk.eagle:library:371" deviceset="GND" device=""/>
+<part name="R5" library="Seeed-Resistor" library_urn="urn:adsk.eagle:library:474" deviceset="SMD-RES-0R-5%-1/16W(0402)" device="" value="0R"/>
+<part name="GND24" library="supply1" library_urn="urn:adsk.eagle:library:371" deviceset="GND" device=""/>
 </parts>
 <sheets>
 <sheet>
 <plain>
+<text x="58.42" y="96.52" size="1.778" layer="97" rot="R90">Bridge to disable CEC</text>
 </plain>
 <instances>
@@
 <instance part="SPDIF" gate="G$1" x="86.36" y="203.2"/>
 <instance part="GND23" gate="1" x="182.88" y="91.44"/>
+<instance part="R5" gate="G$1" x="60.96" y="96.52" rot="R90"/>
+<instance part="GND24" gate="1" x="60.96" y="86.36"/>
 </instances>
 <busses>
@@
 </segment>
 </net>
-<net name="N$2" class="0">
+<net name="A2VDD" class="0">
 <segment>
 <pinref part="U1" gate="A" pin="A2VDD"/>
@@
 </segment>
 </net>
-<net name="N$3" class="0">
+<net name="DVDD" class="0">
 <segment>
 <pinref part="U1" gate="A" pin="DVDD_2"/>
@@
 <pinref part="GND23" gate="1" pin="GND"/>
 </segment>
-</net>
-<net name="N$1" class="0">
+<segment>
+<pinref part="R5" gate="G$1" pin="1"/>
+<pinref part="GND24" gate="1" pin="GND"/>
+<wire x1="60.96" y1="92.71" x2="60.96" y2="88.9" width="0.1524" layer="91"/>
+</segment>
+</net>
+<net name="PVDD" class="0">
 <segment>
 <pinref part="U1" gate="A" pin="PVDD"/>
@@
 </segment>
 </net>
-<net name="N$4" class="0">
+<net name="V1P2" class="0">
 <segment>
 <pinref part="U1" gate="A" pin="V1P2_2"/>
@@
 </segment>
 </net>
-<net name="N$5" class="0">
+<net name="V3P3" class="0">
 <segment>
 <pinref part="U1" gate="A" pin="V3P3"/>
@@
 <pinref part="X1" gate="G$1" pin="OUT"/>
 <pinref part="U1" gate="A" pin="CEC_CLK_I"/>
-<wire x1="50.8" y1="101.6" x2="106.68" y2="101.6" width="0.1524" layer="91"/>
+<wire x1="50.8" y1="101.6" x2="60.96" y2="101.6" width="0.1524" layer="91"/>
+<pinref part="R5" gate="G$1" pin="2"/>
+<wire x1="60.96" y1="101.6" x2="106.68" y2="101.6" width="0.1524" layer="91"/>
+<wire x1="60.96" y1="100.33" x2="60.96" y2="101.6" width="0.1524" layer="91"/>
+<junction x="60.96" y="101.6"/>
 </segment>
 </net>
@@
 </segment>
 </net>
-<net name="N$15" class="0">
+<net name="TXC_P" class="0">
 <segment>
 <pinref part="U3" gate="G$1" pin="TMDS_CK+_SYS"/>
@@
 </segment>
 </net>
-<net name="N$16" class="0">
+<net name="TXC_N" class="0">
 <segment>
 <pinref part="U3" gate="G$1" pin="TMDS_CK-_SYS"/>
@@
 </segment>
 </net>
-<net name="N$17" class="0">
+<net name="TX2_P" class="0">
 <segment>
 <pinref part="U1" gate="A" pin="TX2+"/>
@@
 </segment>
 </net>
-<net name="N$18" class="0">
+<net name="TX2_N" class="0">
 <segment>
 <pinref part="U1" gate="A" pin="TX2-"/>
@@
 </segment>
 </net>
-<net name="N$19" class="0">
+<net name="TX1_P" class="0">
 <segment>
 <pinref part="U1" gate="A" pin="TX1+"/>
@@
 </segment>
 </net>
-<net name="N$20" class="0">
+<net name="TX1_N" class="0">
 <segment>
 <pinref part="U1" gate="A" pin="TX1-"/>
@@
 </segment>
 </net>
-<net name="N$21" class="0">
+<net name="TX0_P" class="0">
 <segment>
 <pinref part="U1" gate="A" pin="TX0+"/>
@@
 </segment>
 </net>
-<net name="N$22" class="0">
+<net name="TX0_N" class="0">
 <segment>
 <pinref part="U1" gate="A" pin="TX0-"/>
@@
 </segment>
 </net>
-<net name="N$28" class="0">
+<net name="AVDD" class="0">
 <segment>
 <pinref part="L1" gate="L" pin="1"/>
